Commit message: feat(flocking): 1. 增加了 flocking 的基础架构   2. 增加了 vswarm_quad 的文件模型

File: gym_pybullet_drones/assets/vswarm_quad/vswarm_quad.urdf (robot description, URDF)
Before this commit: robot cf2, 6 links, 5 joints
Links:
- link base_link: geometry collision cylinder length=.025 radius=.06; visual mesh filename=./cf2.dae scale=1 1 1

File: gym_pybullet_drones/assets/vswarm_quad/vswarm_quad_dae.urdf (robot description, URDF)
Before this commit: robot cf2, 6 links, 5 joints
Links:
- link base_link: geometry collision cylinder length=.025 radius=.06; visual mesh filename=./vswarm_quad.stl scale=0.3 0.3 0.3
