Commit message: feat: 论文答辩前版本

File: gym_pybullet_drones/assets/vswarm_quad/vswarm_quad_dae.urdf (robot description, URDF)
Before this commit: robot cf2, 6 links, 5 joints
Links:
- link base_link: geometry collision cylinder length=.025 radius=.06; visual mesh filename=./vswarm_quad.stl scale=0.7 0.7 0.7
